File: 24V AC SSR Board.brd (EAGLE design)
At the start: 96.5 x 63.2 mm, 41 parts

Commit message: Added new opto-isolators and new custome library
Routing:
- net V-: track 96.0 -> 102.4 mm
- net +24V: track 154.2 -> 149.9 mm, vias 1 -> 0
- net N$24: track 14.5 -> 16.8 mm
Changed lines of the file:
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@@
 <text x="6.985" y="42.545" size="0.889" layer="25">39</text>
 <text x="17.145" y="42.545" size="0.889" layer="25">40</text>
-<rectangle x1="54.61" y1="40.64" x2="62.23" y2="93.98" layer="16"/>
 <text x="5.715" y="58.42" size="0.762" layer="25" rot="R270">http://www.quiller.io</text>
 </plain>
@@
 <contactref element="LED5" pad="A"/>
 <contactref element="D2" pad="C"/>
-<wire x1="66.0654" y1="86.4108" x2="66.675" y2="86.36" width="0" layer="19" extent="1-16"/>
 <wire x1="66.0654" y1="86.1822" x2="66.675" y2="86.36" width="0.254" layer="16"/>
 <wire x1="69.215" y1="85.725" x2="70.485" y2="90.17" width="0.8128" layer="16"/>
@@
 <contactref element="D1" pad="C"/>
 <contactref element="LED4" pad="A"/>
-<wire x1="92.075" y1="57.785" x2="90.17" y2="52.07" width="0.8128" layer="16"/>
-<wire x1="90.17" y1="52.07" x2="93.98" y2="44.45" width="0.8128" layer="16"/>
+<wire x1="90.17" y1="52.07" x2="92.075" y2="53.975" width="0.8128" layer="16"/>
+<wire x1="92.075" y1="53.975" x2="92.075" y2="57.785" width="0.8128" layer="16"/>
+<wire x1="93.98" y1="44.45" x2="93.98" y2="50.165" width="0.8128" layer="16"/>
+<wire x1="93.98" y1="50.165" x2="92.075" y2="52.07" width="0.8128" layer="16"/>
+<wire x1="92.075" y1="52.07" x2="90.17" y2="52.07" width="0.8128" layer="16"/>
 </signal>
 <signal name="GND">
@@
 <wire x1="82.35" y1="64.97" x2="80.645" y2="67.31" width="1.27" layer="16"/>
 <wire x1="80.645" y1="67.31" x2="59.055" y2="67.31" width="1.27" layer="16"/>
-<wire x1="59.055" y1="67.31" x2="59.055" y2="63.5" width="0.4064" layer="16"/>
-<wire x1="59.055" y1="63.5" x2="55.245" y2="59.69" width="0.4064" layer="16"/>
-<wire x1="55.245" y1="59.69" x2="50.8" y2="59.69" width="1.27" layer="16"/>
-<wire x1="50.8" y1="74.93" x2="55.88" y2="74.93" width="1.27" layer="16"/>
-<wire x1="55.88" y1="74.93" x2="55.88" y2="69.215" width="0.4064" layer="16"/>
-<wire x1="55.88" y1="69.215" x2="58.42" y2="66.675" width="0.4064" layer="16"/>
-<wire x1="58.42" y1="66.675" x2="59.055" y2="67.31" width="0.4064" layer="16"/>
-<wire x1="50.8" y1="90.17" x2="57.15" y2="90.17" width="1.27" layer="16"/>
-<wire x1="57.15" y1="90.17" x2="58.42" y2="88.9" width="0.4064" layer="16"/>
-<wire x1="58.42" y1="88.9" x2="58.42" y2="74.93" width="0.4064" layer="16"/>
-<wire x1="58.42" y1="74.93" x2="58.42" y2="66.675" width="0.4064" layer="16"/>
-<wire x1="50.8" y1="44.45" x2="57.15" y2="44.45" width="1.27" layer="16"/>
-<wire x1="57.15" y1="44.45" x2="59.055" y2="46.355" width="0.4064" layer="16"/>
-<wire x1="59.055" y1="46.355" x2="59.055" y2="63.5" width="0.4064" layer="16"/>
+<wire x1="58.7375" y1="66.9925" x2="59.055" y2="67.31" width="0.4064" layer="16"/>
 <wire x1="84.455" y1="57.785" x2="84.455" y2="64.97" width="0.8128" layer="16"/>
 <wire x1="50.8" y1="74.93" x2="48.26" y2="74.93" width="0.8128" layer="16"/>
@@
 <wire x1="50.8" y1="44.45" x2="48.26" y2="44.45" width="0.8128" layer="16"/>
 <wire x1="48.26" y1="44.45" x2="44.45" y2="48.26" width="0.8128" layer="16"/>
-<via x="58.42" y="74.93" extent="1-16" drill="0.8"/>
+<wire x1="50.8" y1="59.69" x2="55.245" y2="59.69" width="1.27" layer="16"/>
+<wire x1="55.245" y1="59.69" x2="58.42" y2="62.865" width="1.27" layer="16"/>
+<wire x1="58.42" y1="62.865" x2="58.42" y2="66.675" width="1.27" layer="16"/>
+<wire x1="58.42" y1="66.675" x2="58.7375" y2="66.9925" width="1.27" layer="16"/>
+<wire x1="50.8" y1="74.93" x2="55.245" y2="74.93" width="1.27" layer="16"/>
+<wire x1="55.245" y1="74.93" x2="58.42" y2="71.755" width="1.27" layer="16"/>
+<wire x1="58.42" y1="71.755" x2="58.42" y2="67.31" width="1.27" layer="16"/>
+<wire x1="58.42" y1="67.31" x2="58.7375" y2="66.9925" width="1.27" layer="16"/>
+<wire x1="48.26" y1="90.17" x2="55.245" y2="90.17" width="1.27" layer="16"/>
+<wire x1="55.245" y1="90.17" x2="58.42" y2="86.995" width="1.27" layer="16"/>
+<wire x1="58.42" y1="86.995" x2="58.42" y2="78.105" width="1.27" layer="16"/>
+<wire x1="58.42" y1="78.105" x2="55.245" y2="74.93" width="1.27" layer="16"/>
+<wire x1="48.26" y1="59.69" x2="54.61" y2="59.69" width="1.27" layer="16"/>
+<wire x1="54.61" y1="59.69" x2="58.42" y2="55.88" width="1.27" layer="16"/>
+<wire x1="58.42" y1="55.88" x2="58.42" y2="47.625" width="1.27" layer="16"/>
+<wire x1="58.42" y1="47.625" x2="55.245" y2="44.45" width="1.27" layer="16"/>
+<wire x1="55.245" y1="44.45" x2="50.8" y2="44.45" width="1.27" layer="16"/>
 </signal>
 <signal name="V-">
@@
 <contactref element="LED6" pad="K"/>
 <contactref element="TERM" pad="2"/>
-<wire x1="80.01" y1="55.245" x2="73.66" y2="60.325" width="0.8128" layer="16"/>
 <wire x1="73.66" y1="60.325" x2="80.01" y2="60.325" width="0.8128" layer="1"/>
 <wire x1="80.01" y1="60.325" x2="87.63" y2="69.97" width="0.8128" layer="1"/>
 <wire x1="87.63" y1="69.97" x2="79.375" y2="71.12" width="0.8128" layer="16"/>
-<wire x1="79.375" y1="71.12" x2="73.025" y2="75.565" width="0.8128" layer="16"/>
 <wire x1="79.375" y1="85.725" x2="79.375" y2="71.12" width="0.8128" layer="16"/>
-<wire x1="79.375" y1="85.725" x2="73.025" y2="90.17" width="0.8128" layer="16"/>
-<wire x1="80.01" y1="55.245" x2="87.63" y2="52.07" width="0.8128" layer="16"/>
-<wire x1="87.63" y1="52.07" x2="83.82" y2="44.45" width="0.8128" layer="16"/>
-<wire x1="83.82" y1="44.45" x2="80.01" y2="40.005" width="0.8128" layer="16"/>
-<wire x1="73.66" y1="45.085" x2="80.01" y2="40.005" width="0.8128" layer="16"/>
+<wire x1="79.375" y1="85.725" x2="79.375" y2="88.265" width="0.8128" layer="16"/>
+<wire x1="79.375" y1="88.265" x2="77.47" y2="90.17" width="0.8128" layer="16"/>
+<wire x1="77.47" y1="90.17" x2="73.025" y2="90.17" width="0.8128" layer="16"/>
+<wire x1="79.375" y1="71.12" x2="79.375" y2="73.66" width="0.8128" layer="16"/>
+<wire x1="79.375" y1="73.66" x2="77.47" y2="75.565" width="0.8128" layer="16"/>
+<wire x1="77.47" y1="75.565" x2="73.025" y2="75.565" width="0.8128" layer="16"/>
+<wire x1="80.01" y1="55.245" x2="80.01" y2="57.15" width="0.8128" layer="16"/>
+<wire x1="80.01" y1="57.15" x2="78.74" y2="58.42" width="0.8128" layer="16"/>
+<wire x1="78.74" y1="58.42" x2="75.565" y2="58.42" width="0.8128" layer="16"/>
+<wire x1="75.565" y1="58.42" x2="73.66" y2="60.325" width="0.8128" layer="16"/>
+<wire x1="80.01" y1="42.545" x2="77.47" y2="45.085" width="0.8128" layer="16"/>
+<wire x1="77.47" y1="45.085" x2="73.66" y2="45.085" width="0.8128" layer="16"/>
+<wire x1="80.01" y1="40.005" x2="80.01" y2="42.545" width="0.8128" layer="16"/>
+<wire x1="80.01" y1="42.545" x2="81.915" y2="44.45" width="0.8128" layer="16"/>
+<wire x1="81.915" y1="44.45" x2="83.82" y2="44.45" width="0.8128" layer="16"/>
+<wire x1="83.82" y1="44.45" x2="83.82" y2="50.165" width="0.8128" layer="16"/>
+<wire x1="83.82" y1="50.165" x2="85.725" y2="52.07" width="0.8128" layer="16"/>
+<wire x1="87.63" y1="52.07" x2="85.725" y2="52.07" width="0.8128" layer="16"/>
+<wire x1="85.725" y1="52.07" x2="82.55" y2="55.245" width="0.8128" layer="16"/>
+<wire x1="82.55" y1="55.245" x2="80.01" y2="55.245" width="0.8128" layer="16"/>
 </signal>
 <signal name="N$1">
@@
 <wire x1="42.545" y1="75.565" x2="39.37" y2="78.74" width="0.8128" layer="1"/>
 </signal>
-<signal name="N$9">
-<via x="58.42" y="44.45" extent="1-16" drill="0.8"/>
-</signal>
-<signal name="N$11">
-<via x="58.42" y="59.69" extent="1-16" drill="0.8"/>
-</signal>
-<signal name="N$13">
-<via x="58.42" y="90.17" extent="1-16" drill="0.8"/>
-</signal>
 </signals>
