File: 24V AC SSR Board_bk.brd (EAGLE design)
At the start: 96.5 x 63.5 mm, 45 parts, among them X1 1751293

Commit message: Cleaned the board layout
Parts:
- removed TRIAC-1, TRIAC-2, TRIAC-3, TRIAC-4: BT134, myhvac:SOT82
- added U$1, U$2, U$3, U$4: BT134, nich:SOT-82
- moved R17 78.5 mm to (11.4, 12.1)
- moved R13 57.6 mm to (24.1, 12.1)
- moved R12 29.0 mm to (41.3, 12.7)
- moved R10 15.3 mm to (21.0, 8.26), turned to 0 degrees
- moved R1 13.4 mm to (59.7, 21.0)
- moved R3 13.1 mm to (45.7, 20.3)
- moved TERM 10.9 mm to (45.7, 4.45)
- moved R11 8.82 mm to (53.3, 12.7)
- moved D1 8.35 mm to (21.6, 4.45), turned to 180 degrees
- moved LED_OUT_A 6.29 mm to (92.1, 9.53), turned to 0 degrees
- moved LED_OUT_Y 6.29 mm to (83.8, 9.53), turned to 0 degrees
- moved LED_OUT_G 5.85 mm to (75.6, 9.53), turned to 0 degrees
- moved LED_OUT_W 5.46 mm to (67.3, 9.53), turned to 0 degrees
- moved D2 5.12 mm to (69.8, 21.0)
- moved R15 5.08 mm to (88.9, 31.8)
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Connections:
- net +24V: now also U$1.P$2, U$2.P$2, U$3.P$2, U$4.P$2; no longer TRIAC-1.2, TRIAC-2.2, TRIAC-3.2, TRIAC-4.2
- net AUX_OUT: now also TERM.4, U$4.P$1; no longer TERM.5, TRIAC-4.1
- net GREEN_OUT: now also TERM.2, U$2.P$1; no longer TERM.3, TRIAC-2.1
- net N$1: now also U$1.P$3; no longer TRIAC-1.3
- net N$3: now also U$4.P$3; no longer TRIAC-4.3
- net N$5: now also U$3.P$3; no longer TRIAC-3.3
- net N$7: now also U$2.P$3; no longer TRIAC-2.3
- net V-: now also TERM.5; no longer TERM.1
- net WHITE_OUT: now also TERM.1, U$1.P$1; no longer TERM.2, TRIAC-1.1
- net YELLOW_OUT: now also TERM.3, U$3.P$1; no longer TERM.4, TRIAC-3.1
Routing:
- net N$30: track 15.8 -> 95.5 mm, vias 0 -> 4
- net N$23: track 20.9 -> 67.6 mm, vias 0 -> 1
- net V-: track 170.5 -> 131.6 mm
- net AUX_OUT: track 96.7 -> 67.9 mm
- net GREEN_OUT: track 61.5 -> 36.1 mm
- net YELLOW_OUT: track 78.2 -> 53.9 mm
- net WHITE_OUT: track 52.4 -> 29.3 mm
- net N$22: track 19.1 -> 41.5 mm, vias 0 -> 1
- net N$14: track 35.4 -> 48.7 mm
- net N$24: track 11.3 -> 24.4 mm
- net +24V: track 104.2 -> 116.5 mm, vias 4 -> 0
- net N$4: track 13.8 -> 24.9 mm
- net N$11: track 28.2 -> 37.0 mm
- net N$9: track 27.2 -> 35.4 mm
- net N$8: track 10.4 -> 18.1 mm
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Other:
- board text added: "1. White Out 2. Green Out 3. Yellow Out"
- board text added: "4. Aux Out 5. 24v Common 6. 24v Hot"
- board text removed: "1N4001"
- board text removed: "40 Pin Connector for Raspberry Pi 2/B+"
- board text removed: "Aux"
- board text removed: "COM"
- board text removed: "Green"
- board text removed: "HOT"
- board text removed: "White"
- board text removed: "Yellow"
